File: 05_design/electrical_schematic/ADAS_electrical/ADAS_schematic.sch (EAGLE design)
At the start: 16 parts, among them SW1 CT10-XXXX-A2, U1 ARDUINO-MEGAFULL, U2 ADAFRUIT_BNO055, U3 SICK_PLS, U4 ESP12E_DEVKIT

Commit message: Changed to single enable
Connections:
- removed net MTR_L_EN: SV1.3, U1.7
- removed net MTR_R_EN: SV2.3, U1.8
- new net MTR_EN: SV1.3, SV2.3, U1.8
Changed lines of the file:
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@@
 </segment>
 </net>
-<net name="MTR_L_EN" class="0">
+<net name="MTR_EN" class="0">
 <segment>
-<wire x1="58.42" y1="154.94" x2="48.26" y2="154.94" width="0.1524" layer="91"/>
-<label x="48.26" y="154.94" size="1.778" layer="95" rot="R180"/>
-<pinref part="U1" gate="G$1" pin="7"/>
+<pinref part="U1" gate="G$1" pin="8"/>
+<wire x1="58.42" y1="152.4" x2="48.26" y2="152.4" width="0.1524" layer="91"/>
+<label x="48.26" y="152.4" size="1.778" layer="95" rot="R180"/>
 </segment>
 <segment>
@@
 <label x="172.72" y="220.98" size="1.778" layer="95" rot="R180"/>
 </segment>
-</net>
-<net name="MTR_R_EN" class="0">
 <segment>
-<wire x1="58.42" y1="152.4" x2="48.26" y2="152.4" width="0.1524" layer="91"/>
-<label x="48.26" y="152.4" size="1.778" layer="95" rot="R180"/>
-<pinref part="U1" gate="G$1" pin="8"/>
-</segment>
-<segment>
